Commit message: selfdriving: added the wheel and caster

File: selfDringing_and_ros2/ros_code/bumperBot_ws/src/bumperbot_description/urdf/bumperbot.urdf.xacro (robot description, xacro)
@@ -1,10 +1,11 @@
 <?xml version="1.0"?>
-<robot xmlns:xacro="http://www.ros.org/wiki/xacro" name="bumperbot">
+<robot name="bumperbot" xmlns:xacro="http://ros.org/wiki/xacro">
+  <!-- Include Gazebo Parameters -->
   <link name="base_footprint"/>
   <link name="base_link">
     <visual>
-      <origin rpy="0 0 0" xyz="0 0 0"/>
+      <origin xyz="0 0 0" rpy="0 0 0" />
       <geometry>
-        <mesh filename="package://bumperbot_description/meshes/base_link.STL"/>
+        <mesh filename="package://bumperbot_description/meshes/base_link.STL" />
       </geometry>
     </visual>
@@ -12,6 +13,63 @@
   <joint name="base_joint" type="fixed">
     <parent link="base_footprint"/>
-    <child link="base_link"/>
-    <origin rpy="0 0 0" xyz="0 0 0.033"/>
+    <child link="base_link" />
+    <origin xyz="0 0 0.033" rpy="0 0 0"/>
+  </joint>
+  <link name="wheel_right_link">
+    <visual>
+      <origin xyz="0 0 0" rpy="1.57 0 0" />
+      <geometry>
+        <mesh filename="package://bumperbot_description/meshes/wheel_right_link.STL" />
+      </geometry>
+    </visual>
+  </link>
+  <joint name="wheel_right_joint" type="continuous">
+    <origin xyz="0 -0.0701101849418637 0" rpy="0 0 0" /> <!-- 0.7mm frame the base link in y axis-->
+    <parent link="base_link" />
+    <child link="wheel_right_link" />
+    <axis xyz="0 1 0" />
+  </joint>
+  <link
+    name="wheel_left_link">
+    <visual>
+      <origin xyz="0 0 0" rpy="-1.57 0 0" />
+      <geometry>
+        <mesh filename="package://bumperbot_description/meshes/wheel_left_link.STL" />
+      </geometry>
+    </visual>
+  </link>
+  <joint name="wheel_left_joint" type="continuous">
+    <origin xyz="0 0.0701101849418642 0" rpy="0 0 0" />
+    <parent link="base_link" />
+    <child link="wheel_left_link" />
+    <axis xyz="0 1 0" />
+  </joint>
+  <link name="caster_front_link">
+    <visual>
+      <origin xyz="0 0 0" rpy="0 0 0" />
+      <geometry>
+        <mesh filename="package://bumperbot_description/meshes/caster_front_link.STL" />
+      </geometry>
+    </visual>
+  </link>
+  <joint name="caster_front_joint" type="fixed">
+    <origin xyz="0.04755 0 -0.0275" rpy="0 0 0" />
+    <parent link="base_link" />
+    <child link="caster_front_link" />
+    <axis xyz="0 0 0" />
+  </joint>
+  <link name="caster_rear_link">
+    <visual>
+      <origin xyz="0 0 0" rpy="0 0 0" />
+      <geometry>
+        <mesh filename="package://bumperbot_description/meshes/caster_rear_link.STL" />
+      </geometry>
+    </visual>
+  </link>
+  <joint name="caster_rear_joint" type="fixed">
+    <origin xyz="-0.04755 0 -0.0275" rpy="0 0 0" />
+    <parent link="base_link" />
+    <child link="caster_rear_link" />
+    <axis xyz="0 0 0" />
   </joint>
 </robot>
